File: left/left.kicad_sch (KiCad schematic)
At the start: 108 parts

Commit message: some state..
Parts:
- removed J?: AudioJack4, symbol Connector:AudioJack4
- removed J? (x2): Conn_01x12, symbol Connector_Generic:Conn_01x12
- removed J?: Conn_01x05, symbol Connector_Generic:Conn_01x05
- added U1: Elite-C, Keebio-Parts:Elite-C, symbol keebio:Elite-C
- added U2: TRRS, symbol keebio:TRRS
- D_0_0, D_0_1, D_0_2, D_0_3, D_0_4, D_0_5, D_0_6: renamed from D?; footprint (none) -> Keebio-Parts:D_SOD-323
- D_1_0, D_1_1, D_1_2, D_1_3, D_1_4, D_1_5, D_2_0, D_2_1, D_2_2, D_2_3, D_2_4, D_2_5, D_3_0, D_3_1, D_3_2, D_3_3, D_3_4, D_3_5, D_4_0, D_4_1, D_4_2, D_4_3, D_4_4, D_5_0, D_5_1: renamed from D?; footprint (none) -> Keebio-Parts:Diode
- L0, L1, L10, L12, L2, L20, L21, L22, L_0_0, L_0_1, L_0_2, L_0_3, L_0_4, L_0_5, L_0_6, L_1_0, L_1_1, L_1_2, L_1_3, L_1_4, L_1_5, L_2_0, L_2_1, L_2_2, L_2_3, L_2_4, L_2_5, L_3_0, L_3_1, L_3_2, L_3_3, L_3_4, L_3_5, L_4_0, L_4_1, L_4_2, L_4_3, L_4_4, L_5_0, L_5_1: renamed from D?; footprint LED_SMD:LED_WS2812B_PLCC4_5.0x5.0mm_P3.2mm -> Keebio-Parts:SK6812-MINI-E
- S_0_0, S_0_1, S_0_2, S_0_3, S_0_4, S_0_5, S_0_6, S_1_1, S_1_2, S_1_3, S_1_4, S_1_5, S_2_1, S_2_2, S_2_3, S_2_4, S_2_5, S_3_1, S_3_2, S_3_3, S_3_4, S_3_5: renamed from SW?; footprint (none) -> MX_Only:MXOnly-1U-Hotswap
- S_1_0, S_4_4: renamed from SW?; footprint (none) -> MX_Only:MXOnly-1.5U-Hotswap
- S_2_0, S_4_3: renamed from SW?; footprint (none) -> MX_Only:MXOnly-1.75U-Hotswap
- S_3_0: renamed from SW?; footprint (none) -> MX_Only:MXOnly-2.25U-Hotswap
- S_4_0, S_4_1, S_4_2, S_5_0, S_5_1: renamed from SW?; footprint (none) -> MX_Only:MXOnly-1.25U-Hotswap
Connections:
- net +5V: now also L22.1 (VDD)
- net GND: now also L22.3 (VSS)
- net row5: now reaches S_5_1.1
- net row5: now also S_5_0.1
- net col3: now reaches D_3_2.1 (K)
- net col3: now also D_0_3.1 (K), D_1_2.1 (K), D_2_2.1 (K), D_4_2.1 (K)
- net row3: now reaches S_3_3.1
- net row3: now also S_3_0.1, S_3_1.1, S_3_2.1, S_3_4.1, S_3_5.1
- net col2: now reaches D_4_1.1 (K)
- net col2: now also D_0_2.1 (K), D_1_1.1 (K), D_2_1.1 (K), D_3_1.1 (K)
- net row4: now reaches S_4_1.1
- net row4: now also S_4_0.1, S_4_2.1, S_4_3.1, S_4_4.1
- net col4: now reaches D_3_3.1 (K)
- net col4: now also D_0_4.1 (K), D_1_3.1 (K), D_2_3.1 (K), D_4_3.1 (K), D_5_0.1 (K)
- net row2: now reaches S_2_0.1
- net row2: now also S_2_1.1, S_2_2.1, S_2_3.1, S_2_4.1, S_2_5.1
- net row1: now reaches S_1_4.1
- net row1: now also S_1_0.1, S_1_1.1, S_1_2.1, S_1_3.1, S_1_5.1
- net col6: now reaches D_4_4.1 (K)
- net col6: now also D_0_6.1 (K), D_1_5.1 (K), D_2_5.1 (K), D_3_5.1 (K), D_5_1.1 (K)
- net col0: now reaches D_0_0.1 (K)
- net col0: now also D_1_0.1 (K), D_2_0.1 (K), D_3_0.1 (K), D_4_0.1 (K)
- net col5: now reaches D_1_4.1 (K)
- net col5: now also D_0_5.1 (K), D_2_4.1 (K), D_3_4.1 (K)
- net row0: now reaches S_0_6.1
- net row0: now also S_0_0.1, S_0_1.1, S_0_2.1, S_0_3.1, S_0_4.1, S_0_5.1
- net col1: now reaches D_0_1.1 (K)
Other:
- moved on the sheet: D_0_1, D_0_2, D_0_3, D_0_4, D_0_5, D_0_6, D_1_0, D_1_1, D_1_2, D_1_3, D_1_4, D_1_5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
